File: Hardware/Avionics-Board.kicad_sch (KiCad schematic)
At the start: 0 parts

Commit message: Day-2
Parts:
- added C3, C4, C5, C6, C7: 100nF, Capacitor_SMD:C_0402_1005Metric, symbol Device:C_Small
- added J1: USB-C, Connector_USB:USB_C_Plug_Molex_105444, symbol Connector:USB_C_Receptacle_USB2.0_14P
- added Module1: ComputeModule5-CM5, CM5IO:Raspberry-Pi-5-Compute-Module, symbol CM5IO:ComputeModule5-CM5
- added U1: ICM-20948, Sensor_Motion:InvenSense_QFN-24_3x3mm_P0.4mm, symbol Sensor_Motion:ICM-20948
- added U2: BMP390, 10LGA_2X2X0p75_BOS, symbol BMP390:BMP390
Connections:
- new net: J1.A4 (VBUS), J1.A9 (VBUS), J1.B4 (VBUS), J1.B9 (VBUS)
- new net: C5.1, U1.10 (REGOUT)
- new net +1V8: C3.2, Module1.88 (+1.8v_(Output)), Module1.90 (+1.8v_(Output)), U1.8 (VDDIO)
- new net +3V3: C4.1, C6.1, C7.1, Module1.84 (+3.3v_(Output)), Module1.86 (+3.3v_(Output)), U1.13 (VDD), U2.1 (VDDIO), U2.10 (VDD)
- new net +5V: Module1.77 (+5v_(Input)), Module1.79 (+5v_(Input)), Module1.81 (+5v_(Input)), Module1.83 (+5v_(Input)), Module1.85 (+5v_(Input)), Module1.87 (+5v_(Input))
- new net CC1: J1.A5 (CC1), Module1.94 (CC1)
- new net CC2: J1.B5 (CC2), Module1.96 (CC2)
- new net CS_BMP: U2.6 (CSB)
- new net CS_IMU: U1.22 (~{CS})
- new net D+: J1.A6 (D+), J1.B6 (D+), Module1.105 (USB2_P)
- new net D-: J1.A7 (D-), J1.B7 (D-), Module1.103 (USB2_N)
- new net GND: C3.1, C4.2, C5.2, C6.2, C7.2, J1.A1 (GND), J1.A12 (GND), J1.B1 (GND), J1.B12 (GND), J1.S1 (SHIELD), Module1.1 (GND), Module1.101 (USB_OTG_ID), Module1.107 (GND), Module1.108 (GND), Module1.113 (GND), Module1.114 (GND), Module1.119 (GND), Module1.120 (GND), Module1.125 (GND), Module1.126 (GND), Module1.13 (GND), Module1.131 (GND), Module1.132 (GND), Module1.138 (GND), Module1.14 (GND), Module1.144 (GND), Module1.149 (HDMI1_CEC), Module1.150 (GND), Module1.155 (GND), Module1.156 (GND), Module1.161 (GND), Module1.162 (GND), Module1.167 (GND), Module1.168 (GND), Module1.173 (GND), Module1.174 (GND), Module1.179 (GND), Module1.180 (GND), Module1.185 (GND), Module1.186 (GND), Module1.191 (GND), Module1.192 (GND), Module1.197 (GND), Module1.198 (GND), Module1.2 (GND), Module1.22 (GND), Module1.23 (GND), Module1.32 (GND), Module1.33 (GND), Module1.42 (GND), Module1.43 (GND), Module1.52 (GND), Module1.53 (GND), Module1.59 (GND), Module1.60 (GND), Module1.65 (GND), Module1.66 (GND), Module1.7 (GND), Module1.71 (GND), Module1.74 (GND), Module1.8 (GND), Module1.98 (GND), U1.11 (FSYNC), U1.18 (GND), U1.20 (GND), U2.3 (VSS), U2.8 (VSS), U2.9 (VSS)
- new net MISO1: Module1.26 (GPIO19), U1.9 (SDO/AD0), U2.5 (SDO)
- new net MOSI1: Module1.27 (GPIO20), U1.24 (SDA/SDI), U2.4 (SDI)
- new net SCLK1: Module1.25 (GPIO21), U1.23 (SCL/SCLK), U2.2 (SCK)
- no-connect marks 0 -> 2

Commit message: Day-3 (Schematic and PCB)
Parts:
- removed Module1: ComputeModule5-CM5, CM5IO:Raspberry-Pi-5-Compute-Module, symbol CM5IO:ComputeModule5-CM5
- added Module1: ComputeModule5-CM5, Avionics-Board:RPi-CM5, symbol RPi-CM5:ComputeModule5-CM5
- U2: footprint 10LGA_2X2X0p75_BOS -> Avionics-Board:BMP390
Connections:
- net +1V8: now also Module1.88 (+1.8v_(Output)), Module1.90 (+1.8v_(Output))
- net +3V3: now also Module1.84 (+3.3v_(Output)), Module1.86 (+3.3v_(Output))
- net +5V: now also Module1.77 (+5v_(Input)), Module1.79 (+5v_(Input)), Module1.81 (+5v_(Input)), Module1.83 (+5v_(Input)), Module1.85 (+5v_(Input)), Module1.87 (+5v_(Input))
- net CC1: now also Module1.94 (CC1)
- net CC2: now also Module1.96 (CC2)
- net D+: now also Module1.105 (USB2_P)
- net D-: now also Module1.103 (USB2_N)
- net GND: now also Module1.1 (GND), Module1.107 (GND), Module1.108 (GND), Module1.113 (GND), Module1.114 (GND), Module1.119 (GND), Module1.120 (GND), Module1.125 (GND), Module1.126 (GND), Module1.13 (GND), Module1.131 (GND), Module1.132 (GND), Module1.138 (GND), Module1.14 (GND), Module1.144 (GND), Module1.149 (HDMI1_CEC), Module1.150 (GND), Module1.155 (GND), Module1.156 (GND), Module1.161 (GND), Module1.162 (GND), Module1.167 (GND), Module1.168 (GND), Module1.173 (GND), Module1.174 (GND), Module1.179 (GND), Module1.180 (GND), Module1.185 (GND), Module1.186 (GND), Module1.191 (GND), Module1.192 (GND), Module1.197 (GND), Module1.198 (GND), Module1.2 (GND), Module1.22 (GND), Module1.23 (GND), Module1.32 (GND), Module1.33 (GND), Module1.42 (GND), Module1.43 (GND), Module1.52 (GND), Module1.53 (GND), Module1.59 (GND), Module1.60 (GND), Module1.65 (GND), Module1.66 (GND), Module1.7 (GND), Module1.71 (GND), Module1.74 (GND), Module1.8 (GND), Module1.98 (GND)
- net MISO1: now also Module1.26 (GPIO19)
- net MOSI1: now also Module1.27 (GPIO20)
- net SCLK1: now also Module1.25 (GPIO21)

Commit message: update
Other:
- company: (none) -> Astralis
- title: (none) -> VikramSat Avionics Board
Changed lines of the file:
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@@
 	(generator_version "9.0")
 	(paper "A4")
+	(title_block
+		(title "VikramSat Avionics Board")
+		(date "17 July 2025")
+		(rev "v0.1")
+		(company "Astralis")
+	)
 	(junction
 		(at 81.28 106.68)
