File: Hardware/Avionics-Board.kicad_sch (KiCad schematic)
At the start: 9 parts, among them J1 USB-C, U1 ICM-20948, U2 BMP390

Commit message: update
Connections:
- net GND: now also Module1.137 (GND)
Changed lines of the file:
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@@
+	)
+	(junction
+		(at 246.38 78.74)
+		(diameter 0)
+		(color 0 0 0 0)
 	)
 	(junction
@@
 	(wire
 		(pts
-			(xy 246.38 71.12) (xy 246.38 93.98)
+			(xy 246.38 71.12) (xy 246.38 78.74)
 		)
 		(stroke
@@
 	(wire
 		(pts
+			(xy 246.38 78.74) (xy 246.38 93.98)
+		)
+		(stroke
+			(width 0)
+			(type default)
+		)
+	)
+	(wire
+		(pts
 			(xy 81.28 83.82) (xy 85.09 83.82)
 		)
@@
 		)
 		(stroke
+			(width 0)
+			(type default)
+		)
+	)
+	(wire
+		(pts
+			(xy 240.03 78.74) (xy 246.38 78.74)
+		)
+		(stroke

Commit message: Day-5
Parts:
- removed U2: BMP390, Avionics-Board:BMP390, symbol BMP390:BMP390
- added U2: BMP-390, easyeda2kicad:LGA-10_L2.0-W2.0-P0.50-BL, symbol easyeda2kicad:BMP390_C5124834
Connections:
- net +3V3: now also U2.1 (VDDIO), U2.10 (VDD)
- net CS_BMP: now also U2.6 (CSB)
- net GND: now also U2.3 (VSS), U2.8 (VSS), U2.9 (VSS)
- net MISO1: now also U2.5 (SDO)
- net MOSI1: now also U2.4 (SDI)
- net SCLK1: now also U2.2 (SCK)
- no-connect marks 2 -> 3
Other:
- moved on the sheet: C6, C7
