File: Hardware/Avionics-Board.kicad_pcb (KiCad board)
At the start: 2 copper layers, 72 x 72 mm, 8 parts, among them U1 ICM-20948, U2 BMP390

Commit message: Day-5
Parts:
- U2: value BMP390 -> BMP-390; footprint Avionics-Board:BMP390 -> easyeda2kicad:LGA-10_L2.0-W2.0-P0.50-BL
- moved C7 0.91 mm to (144.8, 98.3), turned to 90 degrees
- moved C6 0.45 mm to (146.7, 101.0)
- moved U2 0.39 mm to (144.6, 101.0), turned to 180 degrees
Connections:
- Module1 pad 137: unconnected-(Module1B-GND-Pad137) -> GND
